Commit message: Add files search - doesn't work

File: anel_ws/mycobot_ros2_description/urdf/mycobot_320.xacro (robot description, xacro)
@@ -38,5 +38,5 @@
 		<visual>
 			<geometry>
-				<mesh filename="package://mycobot_ros2_description/meshes/mycobot_320_m5_2022/base.dae"/>
+				<mesh filename="file://$(find mycobot_ros2_description)/meshes/mycobot_320_m5_2022/base.dae"/>
 			</geometry>
 			<origin xyz = "0.0 0 -0.03" rpy = "0 0 ${pi/2}"/>
@@ -72,5 +72,5 @@
 			<geometry>
 				<!--Specify the link's visual appearance using the 3D mesh file.-->
-				<mesh filename="package://mycobot_ros2_description/meshes/mycobot_320_m5_2022/link1.dae"/>
+				<mesh filename="file://$(find mycobot_ros2_description)/meshes/mycobot_320_m5_2022/link1.dae"/>
 			</geometry>
 			<!--Define the position and orientation of the visual representation relative to the
@@ -100,5 +100,5 @@
 		<visual>
 			<geometry>
-				<mesh filename="package://mycobot_ros2_description/meshes/mycobot_320_m5_2022/link2.dae"/>
+				<mesh filename="file://$(find mycobot_ros2_description)/meshes/mycobot_320_m5_2022/link2.dae"/>
 			</geometry>
 			<origin xyz = "0.0 0 -0.06096" rpy = " 0 0 ${-pi/2}"/>
@@ -122,5 +122,5 @@
 		<visual>
 		  	<geometry>
-		   		<mesh filename="package://mycobot_ros2_description/meshes/mycobot_320_m5_2022/link3.dae"/>
+		   		<mesh filename="file://$(find mycobot_ros2_description)/meshes/mycobot_320_m5_2022/link3.dae"/>
 		  	</geometry>
 			<origin xyz = "0.0 0 0.03256 " rpy = " 0 ${-pi/2} 0"/>
@@ -144,5 +144,5 @@
 		<visual>
 			<geometry>
-				<mesh filename="package://mycobot_ros2_description/meshes/mycobot_320_m5_2022/link4.dae"/>
+				<mesh filename="file://$(find mycobot_ros2_description)/meshes/mycobot_320_m5_2022/link4.dae"/>
 			</geometry>
 			<origin xyz = "0.0 0 0.03056 " rpy = " 0 ${-pi/2} 0"/>
@@ -166,5 +166,5 @@
 		<visual>
 		  	<geometry>
-				<mesh filename="package://mycobot_ros2_description/meshes/mycobot_320_m5_2022/link5.dae"/>
+				<mesh filename="file://$(find mycobot_ros2_description)/meshes/mycobot_320_m5_2022/link5.dae"/>
 		  	</geometry>
 		  	<origin xyz = "0.0 0 -0.03356 " rpy = "${-pi/2} 0 0"/>
@@ -188,5 +188,5 @@
 		<visual>
 		  	<geometry>
-				<mesh filename="package://mycobot_ros2_description/meshes/mycobot_320_m5_2022/link6.dae"/>
+				<mesh filename="file://$(find mycobot_ros2_description)/meshes/mycobot_320_m5_2022/link6.dae"/>
 		  	</geometry>
 		  	<origin xyz = "0 0.00 -0.038" rpy = "0 0 0"/>
@@ -210,5 +210,5 @@
 		<visual>
 		  	<geometry>
-				<mesh filename="package://mycobot_ros2_description/meshes/mycobot_320_m5_2022/link7.dae"/>
+				<mesh filename="file://$(find mycobot_ros2_description)/meshes/mycobot_320_m5_2022/link7.dae"/>
 		  	</geometry>
 		  	<origin xyz = "0.0 0 -0.012 " rpy = "0 0 0"/>
@@ -232,5 +232,5 @@
 		<visual>
 		  	<geometry>
-				<mesh filename="package://mycobot_ros2_description/meshes/mycobot_320_m5_2022/gripper_base.dae"/>
+				<mesh filename="file://$(find mycobot_ros2_description)/meshes/mycobot_320_m5_2022/gripper_base.dae"/>
 		  	</geometry>
 		  	<origin xyz = "0.0 0.0 -0.012" rpy = "0 0 0"/>
@@ -254,5 +254,5 @@
 		<visual>
 		  	<geometry>
-		  		<mesh filename="package://mycobot_ros2_description/meshes/mycobot_320_m5_2022/gripper_left1.dae"/>
+		  		<mesh filename="file://$(find mycobot_ros2_description)/meshes/mycobot_320_m5_2022/gripper_left1.dae"/>
 		  	</geometry>
 			<origin xyz = "0.039 -0.0133 -0.012 " rpy = " 0 0 0"/>
@@ -276,5 +276,5 @@
 		<visual>
 		  	<geometry>
-		   		<mesh filename="package://mycobot_ros2_description/meshes/mycobot_320_m5_2022/gripper_left2.dae"/>
+		   		<mesh filename="file://$(find mycobot_ros2_description)/meshes/mycobot_320_m5_2022/gripper_left2.dae"/>
 		  	</geometry>
 			<origin xyz = "0.005 -0.0195 -0.012 " rpy = " 0 0 0"/>
@@ -298,5 +298,5 @@
 		<visual>
 		  	<geometry>
-		   		<mesh filename="package://mycobot_ros2_description/meshes/mycobot_320_m5_2022/gripper_left3.dae"/>
+		   		<mesh filename="file://$(find mycobot_ros2_description)/meshes/mycobot_320_m5_2022/gripper_left3.dae"/>
 		  	</geometry>
 		<origin xyz = "0.012 0.0025 -0.012 " rpy = " 0 0 0"/>
@@ -320,5 +320,5 @@
 		<visual>
 			<geometry>
-		   		<mesh filename="package://mycobot_ros2_description/meshes/mycobot_320_m5_2022/gripper_right1.dae"/>
+		   		<mesh filename="file://$(find mycobot_ros2_description)/meshes/mycobot_320_m5_2022/gripper_right1.dae"/>
 		  	</geometry>
 			<origin xyz = "-0.039 -0.0133 -0.012 " rpy = " 0 0 0"/>
@@ -342,5 +342,5 @@
 		<visual>
 			<geometry>
-		   		<mesh filename="package://mycobot_ros2_description/meshes/mycobot_320_m5_2022/gripper_right2.dae"/>
+		   		<mesh filename="file://$(find mycobot_ros2_description)/meshes/mycobot_320_m5_2022/gripper_right2.dae"/>
 		 	</geometry>
 			<origin xyz = "-0.005 -0.0195 -0.012 " rpy = " 0 0 0"/>
@@ -364,5 +364,5 @@
 		<visual>
 			<geometry>
-		   		<mesh filename="package://mycobot_ros2_description/meshes/mycobot_320_m5_2022/gripper_right3.dae"/>
+		   		<mesh filename="file://$(find mycobot_ros2_description)/meshes/mycobot_320_m5_2022/gripper_right3.dae"/>
 			</geometry>
 			<origin xyz = "-0.012 0.0025 -0.012 " rpy = " 0 0 0"/>

Commit message: Change ownership of dae files
- For some reason `package://` is not recognized in XACRO, but absolute
path works

File: anel_ws/mycobot_ros2_description/urdf/mycobot_320.xacro (robot description, xacro)
@@ -38,5 +38,5 @@
 		<visual>
 			<geometry>
-				<mesh filename="file://$(find mycobot_ros2_description)/meshes/mycobot_320_m5_2022/base.dae"/>
+				<mesh filename="file:///home/anel/GitHub/pick_and_place_ros/anel_ws/mycobot_ros2_description/meshes/mycobot_320/base.dae"/>
 			</geometry>
 			<origin xyz = "0.0 0 -0.03" rpy = "0 0 ${pi/2}"/>
@@ -72,5 +72,5 @@
 			<geometry>
 				<!--Specify the link's visual appearance using the 3D mesh file.-->
-				<mesh filename="file://$(find mycobot_ros2_description)/meshes/mycobot_320_m5_2022/link1.dae"/>
+				<mesh filename="file:///home/anel/GitHub/pick_and_place_ros/anel_ws/mycobot_ros2_description/meshes/mycobot_320/link1.dae"/>
 			</geometry>
 			<!--Define the position and orientation of the visual representation relative to the
@@ -100,5 +100,5 @@
 		<visual>
 			<geometry>
-				<mesh filename="file://$(find mycobot_ros2_description)/meshes/mycobot_320_m5_2022/link2.dae"/>
+				<mesh filename="file:///home/anel/GitHub/pick_and_place_ros/anel_ws/mycobot_ros2_description/meshes/mycobot_320/link2.dae"/>
 			</geometry>
 			<origin xyz = "0.0 0 -0.06096" rpy = " 0 0 ${-pi/2}"/>
@@ -122,5 +122,5 @@
 		<visual>
 		  	<geometry>
-		   		<mesh filename="file://$(find mycobot_ros2_description)/meshes/mycobot_320_m5_2022/link3.dae"/>
+		   		<mesh filename="file:///home/anel/GitHub/pick_and_place_ros/anel_ws/mycobot_ros2_description/meshes/mycobot_320/link3.dae"/>
 		  	</geometry>
 			<origin xyz = "0.0 0 0.03256 " rpy = " 0 ${-pi/2} 0"/>
@@ -144,5 +144,5 @@
 		<visual>
 			<geometry>
-				<mesh filename="file://$(find mycobot_ros2_description)/meshes/mycobot_320_m5_2022/link4.dae"/>
+				<mesh filename="file:///home/anel/GitHub/pick_and_place_ros/anel_ws/mycobot_ros2_description/meshes/mycobot_320/link4.dae"/>
 			</geometry>
 			<origin xyz = "0.0 0 0.03056 " rpy = " 0 ${-pi/2} 0"/>
@@ -166,5 +166,5 @@
 		<visual>
 		  	<geometry>
-				<mesh filename="file://$(find mycobot_ros2_description)/meshes/mycobot_320_m5_2022/link5.dae"/>
+				<mesh filename="file:///home/anel/GitHub/pick_and_place_ros/anel_ws/mycobot_ros2_description/meshes/mycobot_320/link5.dae"/>
 		  	</geometry>
 		  	<origin xyz = "0.0 0 -0.03356 " rpy = "${-pi/2} 0 0"/>
@@ -188,5 +188,5 @@
 		<visual>
 		  	<geometry>
-				<mesh filename="file://$(find mycobot_ros2_description)/meshes/mycobot_320_m5_2022/link6.dae"/>
+				<mesh filename="file:///home/anel/GitHub/pick_and_place_ros/anel_ws/mycobot_ros2_description/meshes/mycobot_320/link6.dae"/>
 		  	</geometry>
 		  	<origin xyz = "0 0.00 -0.038" rpy = "0 0 0"/>
@@ -210,5 +210,5 @@
 		<visual>
 		  	<geometry>
-				<mesh filename="file://$(find mycobot_ros2_description)/meshes/mycobot_320_m5_2022/link7.dae"/>
+				<mesh filename="file:///home/anel/GitHub/pick_and_place_ros/anel_ws/mycobot_ros2_description/meshes/mycobot_320/link7.dae"/>
 		  	</geometry>
 		  	<origin xyz = "0.0 0 -0.012 " rpy = "0 0 0"/>
@@ -232,5 +232,5 @@
 		<visual>
 		  	<geometry>
-				<mesh filename="file://$(find mycobot_ros2_description)/meshes/mycobot_320_m5_2022/gripper_base.dae"/>
+				<mesh filename="file:///home/anel/GitHub/pick_and_place_ros/anel_ws/mycobot_ros2_description/meshes/mycobot_320/gripper_base.dae"/>
 		  	</geometry>
 		  	<origin xyz = "0.0 0.0 -0.012" rpy = "0 0 0"/>
@@ -254,5 +254,5 @@
 		<visual>
 		  	<geometry>
-		  		<mesh filename="file://$(find mycobot_ros2_description)/meshes/mycobot_320_m5_2022/gripper_left1.dae"/>
+		  		<mesh filename="file:///home/anel/GitHub/pick_and_place_ros/anel_ws/mycobot_ros2_description/meshes/mycobot_320/gripper_left1.dae"/>
 		  	</geometry>
 			<origin xyz = "0.039 -0.0133 -0.012 " rpy = " 0 0 0"/>
@@ -276,5 +276,5 @@
 		<visual>
 		  	<geometry>
-		   		<mesh filename="file://$(find mycobot_ros2_description)/meshes/mycobot_320_m5_2022/gripper_left2.dae"/>
+		   		<mesh filename="file:///home/anel/GitHub/pick_and_place_ros/anel_ws/mycobot_ros2_description/meshes/mycobot_320/gripper_left2.dae"/>
 		  	</geometry>
 			<origin xyz = "0.005 -0.0195 -0.012 " rpy = " 0 0 0"/>
@@ -287,5 +287,5 @@
 		</collision>
 	</link>
-	<link name="gripper_left3">
+	<link name="gripper_right1">
 		<inertial>
 			<origin xyz="0 0 0.0" rpy="0 0 0"/>
@@ -297,17 +297,17 @@
 		</inertial>
 		<visual>
-		  	<geometry>
-		   		<mesh filename="file://$(find mycobot_ros2_description)/meshes/mycobot_320_m5_2022/gripper_left3.dae"/>
-		  	</geometry>
-		<origin xyz = "0.012 0.0025 -0.012 " rpy = " 0 0 0"/>
-		</visual>
-		<collision>
-		  	<geometry>
-		   		<box size="0.01 0.01 0.01"/>
-		  	</geometry>
-			<origin xyz = "-0.014 0.005 0.005 " rpy = " 0 0 0"/>
-		</collision>
-	</link>
-	<link name="gripper_right1">
+			<geometry>
+		   		<mesh filename="file:///home/anel/GitHub/pick_and_place_ros/anel_ws/mycobot_ros2_description/meshes/mycobot_320/gripper_right1.dae"/>
+		  	</geometry>
+			<origin xyz = "-0.039 -0.0133 -0.012 " rpy = " 0 0 0"/>
+		</visual>
+		<collision>
+		  	<geometry>
+		   		<box size="0.013 0.02 0.015"/>
+		  	</geometry>
+			<origin xyz = "-0.013 0.042 -0.010 " rpy = " 0 0 0"/>
+		</collision>
+	</link>
+	<link name="gripper_right2">
 		<inertial>
 			<origin xyz="0 0 0.0" rpy="0 0 0"/>
@@ -320,16 +320,16 @@
 		<visual>
 			<geometry>
-		   		<mesh filename="file://$(find mycobot_ros2_description)/meshes/mycobot_320_m5_2022/gripper_right1.dae"/>
-		  	</geometry>
-			<origin xyz = "-0.039 -0.0133 -0.012 " rpy = " 0 0 0"/>
-		</visual>
-		<collision>
-		  	<geometry>
-		   		<box size="0.013 0.02 0.015"/>
-		  	</geometry>
-			<origin xyz = "-0.013 0.042 -0.010 " rpy = " 0 0 0"/>
-		</collision>
-	</link>
-	<link name="gripper_right2">
+		   		<mesh filename="file:///home/anel/GitHub/pick_and_place_ros/anel_ws/mycobot_ros2_description/meshes/mycobot_320/gripper_right2.dae"/>
+		 	</geometry>
+			<origin xyz = "-0.005 -0.0195 -0.012 " rpy = " 0 0 0"/>
+		</visual>
+		<collision>
+		  	<geometry>
+		   		<box size="0.02 0.02 0.02"/>
+		  	</geometry>
+			<origin xyz = "0.025 0.0 -0.010 " rpy = " 0 0 0"/>
+		</collision>
+	</link>
+	<link name="gripper_right3">
 		<inertial>
 			<origin xyz="0 0 0.0" rpy="0 0 0"/>
@@ -342,27 +342,5 @@
 		<visual>
 			<geometry>
-		   		<mesh filename="file://$(find mycobot_ros2_description)/meshes/mycobot_320_m5_2022/gripper_right2.dae"/>
-		 	</geometry>
-			<origin xyz = "-0.005 -0.0195 -0.012 " rpy = " 0 0 0"/>
-		</visual>
-		<collision>
-		  	<geometry>
-		   		<box size="0.02 0.02 0.02"/>
-		  	</geometry>
-			<origin xyz = "0.025 0.0 -0.010 " rpy = " 0 0 0"/>
-		</collision>
-	</link>
-	<link name="gripper_right3">
-		<inertial>
-			<origin xyz="0 0 0.0" rpy="0 0 0"/>
-		  	<mass value="0.007"/>
-		  	<inertia
-				ixx="1e-6" ixy="0.0" ixz="0.0"
-				iyy="1e-6" iyz="0.0"
-				izz="1e-6"/>
-		</inertial>
-		<visual>
-			<geometry>
-		   		<mesh filename="file://$(find mycobot_ros2_description)/meshes/mycobot_320_m5_2022/gripper_right3.dae"/>
+		   		<mesh filename="file:///home/anel/GitHub/pick_and_place_ros/anel_ws/mycobot_ros2_description/meshes/mycobot_320/gripper_right3.dae"/>
 			</geometry>
 			<origin xyz = "-0.012 0.0025 -0.012 " rpy = " 0 0 0"/>
