Commit message: Add mesh folder and update URDF for mycobot 320

File: anel_ws/mycobot_ros2_description/urdf/mycobot_320_m5_2022.urdf (robot description, URDF)
Before this commit: robot firefighter, 7 links, 6 joints
Links:
- link base_link: geometry collision mesh filename=package://mycobot_ros2_description/mesh/base.dae; visual mesh filename=package://mycobot_ros2_description/mesh/base.dae
- link link1: geometry collision mesh filename=package://mycobot_ros2_description/mesh/link1.dae; visual mesh filename=package://mycobot_ros2_description/mesh/link1.dae
- link link2: geometry collision mesh filename=package://mycobot_ros2_description/mesh/link2.dae; visual mesh filename=package://mycobot_ros2_description/mesh/link2.dae
- link link3: geometry collision mesh filename=package://mycobot_ros2_description/mesh/link3.dae; visual mesh filename=package://mycobot_ros2_description/mesh/link3.dae
- link link4: geometry collision mesh filename=package://mycobot_ros2_description/mesh/link4.dae; visual mesh filename=package://mycobot_ros2_description/mesh/link4.dae
- link link5: geometry collision mesh filename=package://mycobot_ros2_description/mesh/link5.dae; visual mesh filename=package://mycobot_ros2_description/mesh/link5.dae
- link link6: geometry collision mesh filename=package://mycobot_ros2_description/mesh/link6.dae; visual mesh filename=package://mycobot_ros2_description/mesh/link6.dae
