Commit message: Fix .xacro file of mycobot found by check_urdf

File: anel_ws/mycobot_gazebo/mycobot_320_gazebo.xacro (robot description, xacro)
@@ -15,5 +15,5 @@
 		<visual>
 			<geometry>
-				<mesh filename="file://$(find mycobot_description)/meshes/mycobot_280/base_link.dae"/>
+				<mesh filename="file://$(find mycobot_ros2_description)/meshes/mycobot_280/base_link.dae"/>
 			</geometry>
 			<origin xyz = "0.0 0 -0.03" rpy = "0 0 ${pi/2}"/>
@@ -21,5 +21,5 @@
 		<collision>
 			<geometry>
-				<mesh filename="file://$(find mycobot_description)/meshes/mycobot_280/base_link.dae"/>
+				<mesh filename="file://$(find mycobot_ros2_description)/meshes/mycobot_280/base_link.dae"/>
 			</geometry>
 			<origin xyz = "0.0 0 -0.03" rpy = "0 0 ${pi/2}"/>
@@ -37,5 +37,5 @@
 		<visual>
 			<geometry>
-				<mesh filename="file://$(find mycobot_description)/meshes/mycobot_280/link1.dae"/>
+				<mesh filename="file://$(find mycobot_ros2_description)/meshes/mycobot_280/link1.dae"/>
 			</geometry>
 			<origin xyz = "0.0 0 0 " rpy = " 0 0 ${-pi/2}"/>
@@ -43,5 +43,5 @@
 		<collision>
 			<geometry>
-				<mesh filename="file://$(find mycobot_description)/meshes/mycobot_280/link1.dae"/>
+				<mesh filename="file://$(find mycobot_ros2_description)/meshes/mycobot_280/link1.dae"/>
 			</geometry>
 			<origin xyz = "0.0 0 0.0 " rpy = " 0 0 ${-pi/2}"/>
@@ -59,5 +59,5 @@
 		<visual>
 			<geometry>
-				<mesh filename="file://$(find mycobot_description)/meshes/mycobot_280/link2.dae"/>
+				<mesh filename="file://$(find mycobot_ros2_description)/meshes/mycobot_280/link2.dae"/>
 			</geometry>
 			<origin xyz = "0.0 0 -0.06096" rpy = " 0 0 ${-pi/2}"/>
@@ -65,5 +65,5 @@
 		<collision>
 			<geometry>
-				<mesh filename="file://$(find mycobot_description)/meshes/mycobot_280/link2.dae"/>
+				<mesh filename="file://$(find mycobot_ros2_description)/meshes/mycobot_280/link2.dae"/>
 			</geometry>
 			<origin xyz = "0.0 0 -0.06096" rpy = " 0 0 ${-pi/2}"/>
@@ -81,5 +81,5 @@
 		<visual>
 		  	<geometry>
-		   		<mesh filename="file://$(find mycobot_description)/meshes/mycobot_280/link3.dae"/>
+		   		<mesh filename="file://$(find mycobot_ros2_description)/meshes/mycobot_280/link3.dae"/>
 		  	</geometry>
 			<origin xyz = "0.0 0 0.03256 " rpy = " 0 ${-pi/2} 0"/>
@@ -87,5 +87,5 @@
 		<collision>
 		  	<geometry>
-		   		<mesh filename="file://$(find mycobot_description)/meshes/mycobot_280/link3.dae"/>
+		   		<mesh filename="file://$(find mycobot_ros2_description)/meshes/mycobot_280/link3.dae"/>
 		  	</geometry>
 		  	<origin xyz = "0.00 0 0.03256 " rpy = " 0 ${-pi/2} 0"/>
@@ -103,5 +103,5 @@
 		<visual>
 			<geometry>
-				<mesh filename="file://$(find mycobot_description)/meshes/mycobot_280/link4.dae"/>
+				<mesh filename="file://$(find mycobot_ros2_description)/meshes/mycobot_280/link4.dae"/>
 			</geometry>
 			<origin xyz = "0.0 0 0.03056 " rpy = " 0 ${-pi/2} 0"/>
@@ -109,5 +109,5 @@
 		<collision>
 			<geometry>
-				<mesh filename="file://$(find mycobot_description)/meshes/mycobot_280/link4.dae"/>
+				<mesh filename="file://$(find mycobot_ros2_description)/meshes/mycobot_280/link4.dae"/>
 			</geometry>
 			<origin xyz = "0.0 0 0.03056 " rpy = " 0 ${-pi/2} 0"/>
@@ -125,5 +125,5 @@
 		<visual>
 		  	<geometry>
-				<mesh filename="file://$(find mycobot_description)/meshes/mycobot_280/link5.dae"/>
+				<mesh filename="file://$(find mycobot_ros2_description)/meshes/mycobot_280/link5.dae"/>
 		  	</geometry>
 		  	<origin xyz = "0.0 0 -0.03356 " rpy = "${-pi/2} 0 0"/>
@@ -131,5 +131,5 @@
 		<collision>
 		   	<geometry>
-		   		<mesh filename="file://$(find mycobot_description)/meshes/mycobot_280/link5.dae"/>
+		   		<mesh filename="file://$(find mycobot_ros2_description)/meshes/mycobot_280/link5.dae"/>
 		  	</geometry>
 		  	<origin xyz = "0.0 0 -0.03356 " rpy = "${-pi/2} 0 0"/>
@@ -147,5 +147,5 @@
 		<visual>
 		  	<geometry>
-				<mesh filename="file://$(find mycobot_description)/meshes/mycobot_280/link6.dae"/>
+				<mesh filename="file://$(find mycobot_ros2_description)/meshes/mycobot_280/link6.dae"/>
 		  	</geometry>
 		  	<origin xyz = "0 0.00 -0.038" rpy = "0 0 0"/>
@@ -153,5 +153,5 @@
 		<collision>
 		   	<geometry>
-		   		<mesh filename="file://$(find mycobot_description)/meshes/mycobot_280/link6.dae"/>
+		   		<mesh filename="file://$(find mycobot_ros2_description)/meshes/mycobot_280/link6.dae"/>
 		  	</geometry>
 		  	<origin xyz = "0 0.00 -0.038" rpy = "0 0 0"/>
@@ -169,5 +169,5 @@
 		<visual>
 		  	<geometry>
-				<mesh filename="file://$(find mycobot_description)/meshes/mycobot_280/link7.dae"/>
+				<mesh filename="file://$(find mycobot_ros2_description)/meshes/mycobot_280/link7.dae"/>
 		  	</geometry>
 		  	<origin xyz = "0.0 0 -0.012 " rpy = "0 0 0"/>
@@ -175,5 +175,5 @@
 		<collision>
 		   	<geometry>
-		   		<mesh filename="file://$(find mycobot_description)/meshes/mycobot_280/link7.dae"/>
+		   		<mesh filename="file://$(find mycobot_ros2_description)/meshes/mycobot_280/link7.dae"/>
 		  	</geometry>
 		  	<origin xyz = "0.0 0 -0.012 " rpy = "0 0 0"/>
@@ -191,5 +191,5 @@
 		<visual>
 		  	<geometry>
-				<mesh filename="file://$(find mycobot_description)/meshes/mycobot_280/gripper_base.dae"/>
+				<mesh filename="file://$(find mycobot_ros2_description)/meshes/mycobot_280/gripper_base.dae"/>
 		  	</geometry>
 		  	<origin xyz = "0.0 0.0 -0.012" rpy = "0 0 0"/>
@@ -197,5 +197,5 @@
 		<collision>
 		   	<geometry>
-		   		<mesh filename="file://$(find mycobot_description)/meshes/mycobot_280/gripper_base.dae"/>
+		   		<mesh filename="file://$(find mycobot_ros2_description)/meshes/mycobot_280/gripper_base.dae"/>
 		  	</geometry>
 		  	<origin xyz = "0.0 0.0 -0.012" rpy = "0 0 0"/>
@@ -213,5 +213,5 @@
 		<visual>
 		  	<geometry>
-		  		<mesh filename="file://$(find mycobot_description)/meshes/mycobot_280/gripper_left1.dae"/>
+		  		<mesh filename="file://$(find mycobot_ros2_description)/meshes/mycobot_280/gripper_left1.dae"/>
 		  	</geometry>
 			<origin xyz = "0.039 -0.0133 -0.012 " rpy = " 0 0 0"/>
@@ -219,5 +219,5 @@
 		<collision>
 		  	<geometry>
-		   		<mesh filename="file://$(find mycobot_description)/meshes/mycobot_280/gripper_left1.dae"/>
+		   		<mesh filename="file://$(find mycobot_ros2_description)/meshes/mycobot_280/gripper_left1.dae"/>
 		  	</geometry>
 			<origin xyz = "0.039 -0.0133 -0.012 " rpy = " 0 0 0"/>
@@ -235,5 +235,5 @@
 		<visual>
 		  	<geometry>
-		   		<mesh filename="file://$(find mycobot_description)/meshes/mycobot_280/gripper_left2.dae"/>
+		   		<mesh filename="file://$(find mycobot_ros2_description)/meshes/mycobot_280/gripper_left2.dae"/>
 		  	</geometry>
 			<origin xyz = "0.005 -0.0195 -0.012 " rpy = " 0 0 0"/>
@@ -241,5 +241,5 @@
 		<collision>
 		  	<geometry>
-		   		<mesh filename="file://$(find mycobot_description)/meshes/mycobot_280/gripper_left2.dae"/>
+		   		<mesh filename="file://$(find mycobot_ros2_description)/meshes/mycobot_280/gripper_left2.dae"/>
 		  	</geometry>
 				<origin xyz = "0.005 -0.0195 -0.012 " rpy = " 0 0 0"/>
@@ -257,5 +257,5 @@
 		<visual>
 		  	<geometry>
-		   		<mesh filename="file://$(find mycobot_description)/meshes/mycobot_280/gripper_left3.dae"/>
+		   		<mesh filename="file://$(find mycobot_ros2_description)/meshes/mycobot_280/gripper_left3.dae"/>
 		  	</geometry>
 		<origin xyz = "0.012 0.0025 -0.012 " rpy = " 0 0 0"/>
@@ -263,5 +263,5 @@
 		<collision>
 		  	<geometry>
-		   		<mesh filename="file://$(find mycobot_description)/meshes/mycobot_280/gripper_left3.dae"/>
+		   		<mesh filename="file://$(find mycobot_ros2_description)/meshes/mycobot_280/gripper_left3.dae"/>
 		  	</geometry>
 			<origin xyz = "0.012 0.0025 -0.012" rpy = " 0 0 0"/>
@@ -279,5 +279,5 @@
 		<visual>
 			<geometry>
-		   		<mesh filename="file://$(find mycobot_description)/meshes/mycobot_280/gripper_right1.dae"/>
+		   		<mesh filename="file://$(find mycobot_ros2_description)/meshes/mycobot_280/gripper_right1.dae"/>
 		  	</geometry>
 			<origin xyz = "-0.039 -0.0133 -0.012 " rpy = " 0 0 0"/>
@@ -285,5 +285,5 @@
 		<collision>
 		  	<geometry>
-		   		<mesh filename="file://$(find mycobot_description)/meshes/mycobot_280/gripper_right1.dae"/>
+		   		<mesh filename="file://$(find mycobot_ros2_description)/meshes/mycobot_280/gripper_right1.dae"/>
 		  	</geometry>
 			<origin xyz = "-0.039 -0.0133 -0.012 " rpy = " 0 0 0"/>
@@ -301,5 +301,5 @@
 		<visual>
 			<geometry>
-		   		<mesh filename="file://$(find mycobot_description)/meshes/mycobot_280/gripper_right2.dae"/>
+		   		<mesh filename="file://$(find mycobot_ros2_description)/meshes/mycobot_280/gripper_right2.dae"/>
 		 	</geometry>
 			<origin xyz = "-0.005 -0.0195 -0.012 " rpy = " 0 0 0"/>
@@ -307,5 +307,5 @@
 		<collision>
 		  	<geometry>
-		   		<mesh filename="file://$(find mycobot_description)/meshes/mycobot_280/gripper_right2.dae"/>
+		   		<mesh filename="file://$(find mycobot_ros2_description)/meshes/mycobot_280/gripper_right2.dae"/>
 		  	</geometry>
 			<origin xyz = "-0.005 -0.0195 -0.012 " rpy = " 0 0 0"/>
@@ -323,5 +323,5 @@
 		<visual>
 			<geometry>
-		   		<mesh filename="file://$(find mycobot_description)/meshes/mycobot_280/gripper_right3.dae"/>
+		   		<mesh filename="file://$(find mycobot_ros2_description)/meshes/mycobot_280/gripper_right3.dae"/>
 			</geometry>
 			<origin xyz = "-0.012 0.0025 -0.012 " rpy = " 0 0 0"/>
@@ -329,5 +329,5 @@
 		<collision>
 		  	<geometry>
-		   		<mesh filename="file://$(find mycobot_description)/meshes/mycobot_280/gripper_right3.dae"/>
+		   		<mesh filename="file://$(find mycobot_ros2_description)/meshes/mycobot_280/gripper_right3.dae"/>
 		  	</geometry>
 			<origin xyz = "-0.012 0.0025 -0.012" rpy = " 0 0 0"/>
