Commit message: Convert xacro to URDF to sdf and import ot Gazebo - works, but not nice

File: anel_ws/mycobot_gazebo/mycobot_320_gazebo.xacro (robot description, xacro)
@@ -15,5 +15,5 @@
 		<visual>
 			<geometry>
-				<mesh filename="file://$(find mycobot_ros2_description)/meshes/mycobot_280/base_link.dae"/>
+				<mesh filename="file://$(find mycobot_ros2_description)/mesh/base_link.dae"/>
 			</geometry>
 			<origin xyz = "0.0 0 -0.03" rpy = "0 0 ${pi/2}"/>
@@ -21,5 +21,5 @@
 		<collision>
 			<geometry>
-				<mesh filename="file://$(find mycobot_ros2_description)/meshes/mycobot_280/base_link.dae"/>
+				<mesh filename="file://$(find mycobot_ros2_description)/mesh/base_link.dae"/>
 			</geometry>
 			<origin xyz = "0.0 0 -0.03" rpy = "0 0 ${pi/2}"/>
@@ -37,5 +37,5 @@
 		<visual>
 			<geometry>
-				<mesh filename="file://$(find mycobot_ros2_description)/meshes/mycobot_280/link1.dae"/>
+				<mesh filename="file://$(find mycobot_ros2_description)/mesh/link1.dae"/>
 			</geometry>
 			<origin xyz = "0.0 0 0 " rpy = " 0 0 ${-pi/2}"/>
@@ -43,5 +43,5 @@
 		<collision>
 			<geometry>
-				<mesh filename="file://$(find mycobot_ros2_description)/meshes/mycobot_280/link1.dae"/>
+				<mesh filename="file://$(find mycobot_ros2_description)/mesh/link1.dae"/>
 			</geometry>
 			<origin xyz = "0.0 0 0.0 " rpy = " 0 0 ${-pi/2}"/>
@@ -59,5 +59,5 @@
 		<visual>
 			<geometry>
-				<mesh filename="file://$(find mycobot_ros2_description)/meshes/mycobot_280/link2.dae"/>
+				<mesh filename="file://$(find mycobot_ros2_description)/mesh/link2.dae"/>
 			</geometry>
 			<origin xyz = "0.0 0 -0.06096" rpy = " 0 0 ${-pi/2}"/>
@@ -65,5 +65,5 @@
 		<collision>
 			<geometry>
-				<mesh filename="file://$(find mycobot_ros2_description)/meshes/mycobot_280/link2.dae"/>
+				<mesh filename="file://$(find mycobot_ros2_description)/mesh/link2.dae"/>
 			</geometry>
 			<origin xyz = "0.0 0 -0.06096" rpy = " 0 0 ${-pi/2}"/>
@@ -81,5 +81,5 @@
 		<visual>
 		  	<geometry>
-		   		<mesh filename="file://$(find mycobot_ros2_description)/meshes/mycobot_280/link3.dae"/>
+		   		<mesh filename="file://$(find mycobot_ros2_description)/mesh/link3.dae"/>
 		  	</geometry>
 			<origin xyz = "0.0 0 0.03256 " rpy = " 0 ${-pi/2} 0"/>
@@ -87,5 +87,5 @@
 		<collision>
 		  	<geometry>
-		   		<mesh filename="file://$(find mycobot_ros2_description)/meshes/mycobot_280/link3.dae"/>
+		   		<mesh filename="file://$(find mycobot_ros2_description)/mesh/link3.dae"/>
 		  	</geometry>
 		  	<origin xyz = "0.00 0 0.03256 " rpy = " 0 ${-pi/2} 0"/>
@@ -103,5 +103,5 @@
 		<visual>
 			<geometry>
-				<mesh filename="file://$(find mycobot_ros2_description)/meshes/mycobot_280/link4.dae"/>
+				<mesh filename="file://$(find mycobot_ros2_description)/mesh/link4.dae"/>
 			</geometry>
 			<origin xyz = "0.0 0 0.03056 " rpy = " 0 ${-pi/2} 0"/>
@@ -109,5 +109,5 @@
 		<collision>
 			<geometry>
-				<mesh filename="file://$(find mycobot_ros2_description)/meshes/mycobot_280/link4.dae"/>
+				<mesh filename="file://$(find mycobot_ros2_description)/mesh/link4.dae"/>
 			</geometry>
 			<origin xyz = "0.0 0 0.03056 " rpy = " 0 ${-pi/2} 0"/>
@@ -125,5 +125,5 @@
 		<visual>
 		  	<geometry>
-				<mesh filename="file://$(find mycobot_ros2_description)/meshes/mycobot_280/link5.dae"/>
+				<mesh filename="file://$(find mycobot_ros2_description)/mesh/link5.dae"/>
 		  	</geometry>
 		  	<origin xyz = "0.0 0 -0.03356 " rpy = "${-pi/2} 0 0"/>
@@ -131,5 +131,5 @@
 		<collision>
 		   	<geometry>
-		   		<mesh filename="file://$(find mycobot_ros2_description)/meshes/mycobot_280/link5.dae"/>
+		   		<mesh filename="file://$(find mycobot_ros2_description)/mesh/link5.dae"/>
 		  	</geometry>
 		  	<origin xyz = "0.0 0 -0.03356 " rpy = "${-pi/2} 0 0"/>
@@ -147,5 +147,5 @@
 		<visual>
 		  	<geometry>
-				<mesh filename="file://$(find mycobot_ros2_description)/meshes/mycobot_280/link6.dae"/>
+				<mesh filename="file://$(find mycobot_ros2_description)/mesh/link6.dae"/>
 		  	</geometry>
 		  	<origin xyz = "0 0.00 -0.038" rpy = "0 0 0"/>
@@ -153,10 +153,10 @@
 		<collision>
 		   	<geometry>
-		   		<mesh filename="file://$(find mycobot_ros2_description)/meshes/mycobot_280/link6.dae"/>
+		   		<mesh filename="file://$(find mycobot_ros2_description)/mesh/link6.dae"/>
 		  	</geometry>
 		  	<origin xyz = "0 0.00 -0.038" rpy = "0 0 0"/>
 		</collision>
 	</link>
-	<link name="link6_flange">
+	<!-- <link name="link6_flange">
 		<inertial>
 			<origin xyz="0 0 0.0" rpy="0 0 0"/>
@@ -169,5 +169,5 @@
 		<visual>
 		  	<geometry>
-				<mesh filename="file://$(find mycobot_ros2_description)/meshes/mycobot_280/link7.dae"/>
+				<mesh filename="file://$(find mycobot_ros2_description)/mesh/link7.dae"/>
 		  	</geometry>
 		  	<origin xyz = "0.0 0 -0.012 " rpy = "0 0 0"/>
@@ -175,10 +175,10 @@
 		<collision>
 		   	<geometry>
-		   		<mesh filename="file://$(find mycobot_ros2_description)/meshes/mycobot_280/link7.dae"/>
+		   		<mesh filename="file://$(find mycobot_ros2_description)/mesh/link7.dae"/>
 		  	</geometry>
 		  	<origin xyz = "0.0 0 -0.012 " rpy = "0 0 0"/>
 		</collision>
-	</link>
-	<link name="gripper_base">
+	</link> -->
+	<!-- <link name="gripper_base">
 		<inertial>
 			<origin xyz="0 0 0.0" rpy="0 0 0"/>
@@ -191,5 +191,5 @@
 		<visual>
 		  	<geometry>
-				<mesh filename="file://$(find mycobot_ros2_description)/meshes/mycobot_280/gripper_base.dae"/>
+				<mesh filename="file://$(find mycobot_ros2_description)/mesh/gripper_base.dae"/>
 		  	</geometry>
 		  	<origin xyz = "0.0 0.0 -0.012" rpy = "0 0 0"/>
@@ -197,5 +197,5 @@
 		<collision>
 		   	<geometry>
-		   		<mesh filename="file://$(find mycobot_ros2_description)/meshes/mycobot_280/gripper_base.dae"/>
+		   		<mesh filename="file://$(find mycobot_ros2_description)/mesh/gripper_base.dae"/>
 		  	</geometry>
 		  	<origin xyz = "0.0 0.0 -0.012" rpy = "0 0 0"/>
@@ -213,5 +213,5 @@
 		<visual>
 		  	<geometry>
-		  		<mesh filename="file://$(find mycobot_ros2_description)/meshes/mycobot_280/gripper_left1.dae"/>
+		  		<mesh filename="file://$(find mycobot_ros2_description)/mesh/gripper_left1.dae"/>
 		  	</geometry>
 			<origin xyz = "0.039 -0.0133 -0.012 " rpy = " 0 0 0"/>
@@ -219,5 +219,5 @@
 		<collision>
 		  	<geometry>
-		   		<mesh filename="file://$(find mycobot_ros2_description)/meshes/mycobot_280/gripper_left1.dae"/>
+		   		<mesh filename="file://$(find mycobot_ros2_description)/mesh/gripper_left1.dae"/>
 		  	</geometry>
 			<origin xyz = "0.039 -0.0133 -0.012 " rpy = " 0 0 0"/>
@@ -235,5 +235,5 @@
 		<visual>
 		  	<geometry>
-		   		<mesh filename="file://$(find mycobot_ros2_description)/meshes/mycobot_280/gripper_left2.dae"/>
+		   		<mesh filename="file://$(find mycobot_ros2_description)/mesh/gripper_left2.dae"/>
 		  	</geometry>
 			<origin xyz = "0.005 -0.0195 -0.012 " rpy = " 0 0 0"/>
@@ -241,5 +241,5 @@
 		<collision>
 		  	<geometry>
-		   		<mesh filename="file://$(find mycobot_ros2_description)/meshes/mycobot_280/gripper_left2.dae"/>
+		   		<mesh filename="file://$(find mycobot_ros2_description)/mesh/gripper_left2.dae"/>
 		  	</geometry>
 				<origin xyz = "0.005 -0.0195 -0.012 " rpy = " 0 0 0"/>
@@ -257,5 +257,5 @@
 		<visual>
 		  	<geometry>
-		   		<mesh filename="file://$(find mycobot_ros2_description)/meshes/mycobot_280/gripper_left3.dae"/>
+		   		<mesh filename="file://$(find mycobot_ros2_description)/mesh/gripper_left3.dae"/>
 		  	</geometry>
 		<origin xyz = "0.012 0.0025 -0.012 " rpy = " 0 0 0"/>
@@ -263,10 +263,10 @@
 		<collision>
 		  	<geometry>
-		   		<mesh filename="file://$(find mycobot_ros2_description)/meshes/mycobot_280/gripper_left3.dae"/>
+		   		<mesh filename="file://$(find mycobot_ros2_description)/mesh/gripper_left3.dae"/>
 		  	</geometry>
 			<origin xyz = "0.012 0.0025 -0.012" rpy = " 0 0 0"/>
 		</collision>
-	</link>
-	<link name="gripper_right1">
+	</link> -->
+	<!-- <link name="gripper_right1">
 		<inertial>
 			<origin xyz="0 0 0.0" rpy="0 0 0"/>
@@ -279,5 +279,5 @@
 		<visual>
 			<geometry>
-		   		<mesh filename="file://$(find mycobot_ros2_description)/meshes/mycobot_280/gripper_right1.dae"/>
+		   		<mesh filename="file://$(find mycobot_ros2_description)/mesh/gripper_right1.dae"/>
 		  	</geometry>
 			<origin xyz = "-0.039 -0.0133 -0.012 " rpy = " 0 0 0"/>
@@ -285,5 +285,5 @@
 		<collision>
 		  	<geometry>
-		   		<mesh filename="file://$(find mycobot_ros2_description)/meshes/mycobot_280/gripper_right1.dae"/>
+		   		<mesh filename="file://$(find mycobot_ros2_description)/mesh/gripper_right1.dae"/>
 		  	</geometry>
 			<origin xyz = "-0.039 -0.0133 -0.012 " rpy = " 0 0 0"/>
@@ -301,5 +301,5 @@
 		<visual>
 			<geometry>
-		   		<mesh filename="file://$(find mycobot_ros2_description)/meshes/mycobot_280/gripper_right2.dae"/>
+		   		<mesh filename="file://$(find mycobot_ros2_description)/mesh/gripper_right2.dae"/>
 		 	</geometry>
 			<origin xyz = "-0.005 -0.0195 -0.012 " rpy = " 0 0 0"/>
@@ -307,5 +307,5 @@
 		<collision>
 		  	<geometry>
-		   		<mesh filename="file://$(find mycobot_ros2_description)/meshes/mycobot_280/gripper_right2.dae"/>
+		   		<mesh filename="file://$(find mycobot_ros2_description)/mesh/gripper_right2.dae"/>
 		  	</geometry>
 			<origin xyz = "-0.005 -0.0195 -0.012 " rpy = " 0 0 0"/>
@@ -323,5 +323,5 @@
 		<visual>
 			<geometry>
-		   		<mesh filename="file://$(find mycobot_ros2_description)/meshes/mycobot_280/gripper_right3.dae"/>
+		   		<mesh filename="file://$(find mycobot_ros2_description)/mesh/gripper_right3.dae"/>
 			</geometry>
 			<origin xyz = "-0.012 0.0025 -0.012 " rpy = " 0 0 0"/>
@@ -329,9 +329,10 @@
 		<collision>
 		  	<geometry>
-		   		<mesh filename="file://$(find mycobot_ros2_description)/meshes/mycobot_280/gripper_right3.dae"/>
+		   		<mesh filename="file://$(find mycobot_ros2_description)/mesh/gripper_right3.dae"/>
 		  	</geometry>
 			<origin xyz = "-0.012 0.0025 -0.012" rpy = " 0 0 0"/>
 		</collision>
 	</link>
+   -->
 	<joint name="virtual_joint" type="fixed">
 		<parent link="world"/>
@@ -384,5 +385,5 @@
         <dynamics damping="0.01" friction="0.005"/>
 	</joint>
-	<joint name="link6_to_link6flange" type="revolute">
+	<!-- <joint name="link6_to_link6flange" type="revolute">
 		<axis xyz=" 0 0 1"/>
 		<limit effort = "${effort}" lower = "-3.05" upper = "3.05" velocity = "${velocity}"/>
@@ -396,5 +397,6 @@
 		<child link="gripper_base"/>
 		<origin xyz= "0 0 0.034" rpy = "1.579 0 0"/>
-	</joint>
+	</joint> -->
+<!--
 	<joint name="gripper_controller" type="revolute">
 		<axis xyz="0 0 1"/>
@@ -449,5 +451,5 @@
 		<mimic joint="gripper_controller" multiplier="1.0" offset="0" />
         <dynamics damping="0.01" friction="0.005"/>
-	</joint>
+	</joint> -->
     <gazebo>
         <plugin filename="ignition-gazebo-joint-state-publisher-system" name="ignition::gazebo::systems::JointStatePublisher">

File: anel_ws/mycobot_ros2_description/urdf/mycobot_320.xacro (robot description, xacro)
@@ -38,5 +38,5 @@
 		<visual>
 			<geometry>
-				<mesh filename="file:///home/anel/GitHub/pick_and_place_ros/anel_ws/mycobot_ros2_description/meshes/mycobot_320/base.dae"/>
+				<mesh filename="file:///home/anel/GitHub/pick_and_place_ros/anel_ws/mycobot_ros2_description/mesh/mycobot_320/base.dae"/>
 			</geometry>
 			<origin xyz = "0.0 0 -0.03" rpy = "0 0 ${pi/2}"/>
@@ -72,5 +72,5 @@
 			<geometry>
 				<!--Specify the link's visual appearance using the 3D mesh file.-->
-				<mesh filename="file:///home/anel/GitHub/pick_and_place_ros/anel_ws/mycobot_ros2_description/meshes/mycobot_320/link1.dae"/>
+				<mesh filename="file:///home/anel/GitHub/pick_and_place_ros/anel_ws/mycobot_ros2_description/mesh/mycobot_320/link1.dae"/>
 			</geometry>
 			<!--Define the position and orientation of the visual representation relative to the
@@ -100,5 +100,5 @@
 		<visual>
 			<geometry>
-				<mesh filename="file:///home/anel/GitHub/pick_and_place_ros/anel_ws/mycobot_ros2_description/meshes/mycobot_320/link2.dae"/>
+				<mesh filename="file:///home/anel/GitHub/pick_and_place_ros/anel_ws/mycobot_ros2_description/mesh/mycobot_320/link2.dae"/>
 			</geometry>
 			<origin xyz = "0.0 0 -0.06096" rpy = " 0 0 ${-pi/2}"/>
@@ -122,5 +122,5 @@
 		<visual>
 		  	<geometry>
-		   		<mesh filename="file:///home/anel/GitHub/pick_and_place_ros/anel_ws/mycobot_ros2_description/meshes/mycobot_320/link3.dae"/>
+		   		<mesh filename="file:///home/anel/GitHub/pick_and_place_ros/anel_ws/mycobot_ros2_description/mesh/mycobot_320/link3.dae"/>
 		  	</geometry>
 			<origin xyz = "0.0 0 0.03256 " rpy = " 0 ${-pi/2} 0"/>
@@ -144,5 +144,5 @@
 		<visual>
 			<geometry>
-				<mesh filename="file:///home/anel/GitHub/pick_and_place_ros/anel_ws/mycobot_ros2_description/meshes/mycobot_320/link4.dae"/>
+				<mesh filename="file:///home/anel/GitHub/pick_and_place_ros/anel_ws/mycobot_ros2_description/mesh/mycobot_320/link4.dae"/>
 			</geometry>
 			<origin xyz = "0.0 0 0.03056 " rpy = " 0 ${-pi/2} 0"/>
@@ -166,5 +166,5 @@
 		<visual>
 		  	<geometry>
-				<mesh filename="file:///home/anel/GitHub/pick_and_place_ros/anel_ws/mycobot_ros2_description/meshes/mycobot_320/link5.dae"/>
+				<mesh filename="file:///home/anel/GitHub/pick_and_place_ros/anel_ws/mycobot_ros2_description/mesh/mycobot_320/link5.dae"/>
 		  	</geometry>
 		  	<origin xyz = "0.0 0 -0.03356 " rpy = "${-pi/2} 0 0"/>
@@ -188,5 +188,5 @@
 		<visual>
 		  	<geometry>
-				<mesh filename="file:///home/anel/GitHub/pick_and_place_ros/anel_ws/mycobot_ros2_description/meshes/mycobot_320/link6.dae"/>
+				<mesh filename="file:///home/anel/GitHub/pick_and_place_ros/anel_ws/mycobot_ros2_description/mesh/mycobot_320/link6.dae"/>
 		  	</geometry>
 		  	<origin xyz = "0 0.00 -0.038" rpy = "0 0 0"/>
@@ -199,5 +199,5 @@
 		</collision>
 	</link>
-	<link name="link6_flange">
+	<!-- <link name="link6_flange">
 		<inertial>
 			<origin xyz="0 0 0.0" rpy="0 0 0"/>
@@ -210,5 +210,5 @@
 		<visual>
 		  	<geometry>
-				<mesh filename="file:///home/anel/GitHub/pick_and_place_ros/anel_ws/mycobot_ros2_description/meshes/mycobot_320/link7.dae"/>
+				<mesh filename="file:///home/anel/GitHub/pick_and_place_ros/anel_ws/mycobot_ros2_description/mesh/mycobot_320/link7.dae"/>
 		  	</geometry>
 		  	<origin xyz = "0.0 0 -0.012 " rpy = "0 0 0"/>
@@ -220,6 +220,6 @@
 		  	<origin xyz = "0 0.00 0.0" rpy = "0 0 0"/>
 		</collision>
-	</link>
-	<link name="gripper_base">
+	</link> -->
+	<!-- <link name="gripper_base">
 		<inertial>
 			<origin xyz="0 0 0.0" rpy="0 0 0"/>
@@ -232,5 +232,5 @@
 		<visual>
 		  	<geometry>
-				<mesh filename="file:///home/anel/GitHub/pick_and_place_ros/anel_ws/mycobot_ros2_description/meshes/mycobot_320/gripper_base.dae"/>
+				<mesh filename="file:///home/anel/GitHub/pick_and_place_ros/anel_ws/mycobot_ros2_description/mesh/mycobot_320/gripper_base.dae"/>
 		  	</geometry>
 		  	<origin xyz = "0.0 0.0 -0.012" rpy = "0 0 0"/>
@@ -254,5 +254,5 @@
 		<visual>
 		  	<geometry>
-		  		<mesh filename="file:///home/anel/GitHub/pick_and_place_ros/anel_ws/mycobot_ros2_description/meshes/mycobot_320/gripper_left1.dae"/>
+		  		<mesh filename="file:///home/anel/GitHub/pick_and_place_ros/anel_ws/mycobot_ros2_description/mesh/mycobot_320/gripper_left1.dae"/>
 		  	</geometry>
 			<origin xyz = "0.039 -0.0133 -0.012 " rpy = " 0 0 0"/>
@@ -276,5 +276,5 @@
 		<visual>
 		  	<geometry>
-		   		<mesh filename="file:///home/anel/GitHub/pick_and_place_ros/anel_ws/mycobot_ros2_description/meshes/mycobot_320/gripper_left2.dae"/>
+		   		<mesh filename="file:///home/anel/GitHub/pick_and_place_ros/anel_ws/mycobot_ros2_description/mesh/mycobot_320/gripper_left2.dae"/>
 		  	</geometry>
 			<origin xyz = "0.005 -0.0195 -0.012 " rpy = " 0 0 0"/>
@@ -298,5 +298,5 @@
 		<visual>
 			<geometry>
-		   		<mesh filename="file:///home/anel/GitHub/pick_and_place_ros/anel_ws/mycobot_ros2_description/meshes/mycobot_320/gripper_right1.dae"/>
+		   		<mesh filename="file:///home/anel/GitHub/pick_and_place_ros/anel_ws/mycobot_ros2_description/mesh/mycobot_320/gripper_right1.dae"/>
 		  	</geometry>
 			<origin xyz = "-0.039 -0.0133 -0.012 " rpy = " 0 0 0"/>
@@ -320,5 +320,5 @@
 		<visual>
 			<geometry>
-		   		<mesh filename="file:///home/anel/GitHub/pick_and_place_ros/anel_ws/mycobot_ros2_description/meshes/mycobot_320/gripper_right2.dae"/>
+		   		<mesh filename="file:///home/anel/GitHub/pick_and_place_ros/anel_ws/mycobot_ros2_description/mesh/mycobot_320/gripper_right2.dae"/>
 		 	</geometry>
 			<origin xyz = "-0.005 -0.0195 -0.012 " rpy = " 0 0 0"/>
@@ -342,5 +342,5 @@
 		<visual>
 			<geometry>
-		   		<mesh filename="file:///home/anel/GitHub/pick_and_place_ros/anel_ws/mycobot_ros2_description/meshes/mycobot_320/gripper_right3.dae"/>
+		   		<mesh filename="file:///home/anel/GitHub/pick_and_place_ros/anel_ws/mycobot_ros2_description/mesh/mycobot_320/gripper_right3.dae"/>
 			</geometry>
 			<origin xyz = "-0.012 0.0025 -0.012 " rpy = " 0 0 0"/>
@@ -353,4 +353,5 @@
 		</collision>
 	</link>
+   -->
 	<!-- ********** JOINTS ********** -->
 	<!-- Attach the robot base to the world frame with no initial offset or rotation. -->
@@ -420,5 +421,5 @@
 		<origin xyz= "0 -0.07318 0" rpy = "${pi/2} ${-pi/2} 0"/>
 	</joint>
-	<joint name="link6_to_link6flange" type="revolute">
+	<!-- <joint name="link6_to_link6flange" type="revolute">
 		<axis xyz=" 0 0 1"/>
 		<limit effort = "${effort}" lower = "-3.05" upper = "3.05" velocity = "${velocity}"/>
@@ -438,9 +439,9 @@
 		<child link="gripper_left3"/>
 		<origin xyz= "-0.012 0.005 0" rpy = "0 0 0"/>
-	</joint>
+	</joint> -->
 	<!-- The mimic element means this joint will follow the movements of the
 		gripper_controller joint.
 	-->
-	<joint name="gripper_base_to_gripper_left2" type="revolute">
+	<!-- <joint name="gripper_base_to_gripper_left2" type="revolute">
 		<axis xyz="0 0 1"/>
 		<limit effort = "${effort}" lower = "-0.8" upper = "0.5" velocity = "${velocity}"/>
@@ -481,4 +482,4 @@
 		<origin xyz= "0.027 0.016 0" rpy = "0 0 0"/>
 		<mimic joint="gripper_controller" multiplier="1.0" offset="0" />
-	</joint>
+	</joint> -->
 </robot>
