Commit message: FIx controller loading, but still problem with command for movement
- Seems like `/joint_states` are not receiving the angles published by
  `arm_controller/joint_trajectory`
- What I'm missing?

File: my_project/src/mycobot_description/xacro/macro.gazebo_config_ros2_control.xacro (robot description, xacro)
@@ -1,6 +1,5 @@
 <?xml version="1.0" ?>
 <robot xmlns:xacro="http://wiki.ros.org/xacro">
-    <xacro:macro name="config_ctr_gazebo">
-    <!-- I need this for ROS2 control
+    <!-- I need this for ROS2 control - hardware interface
          it needs <plugin> - parses the ros2_control tags and loads the appropriate hardware interfaces and controller manager,
          and <joint> tags including the robot controllers: commands and states.
@@ -15,8 +14,13 @@
     <!-- I created this file, it was NOT available in the original mycobot repo -->
     <!-- but it is here https://github.com/automaticaddison/mycobot_ros2/blob/main/mycobot_gazebo/urdf/ros2_control/gazebo/mycobot_280_ros2_control.xacro -->
+    <!-- [Err] [SystemLoader.cc:92] Failed to load system plugin [gz_ros2_control-system] : Could not find shared library. -->
+    <!-- Gazebo Fortress and Humble are supported from pacakge `ros-humble-ign-ros2-control` https://github.com/ros-controls/gz_ros2_control/tree/humble-->
+    <!-- We need to build the gz_ros2_control for Harmonic only from source https://github.com/ros-controls/gz_ros2_control/tree/iron and switch to ROS2 Iron
+    -->
     <ros2_control name="GazeboSimSystem" type="system">
         <hardware>
             <plugin>gz_ros2_control/GazeboSimSystem</plugin>
         </hardware>
+        <!-- command - controlling position; state - reading the position,velocity, effort -->
         <joint name="joint2_to_joint1">
             <command_interface name="position">
@@ -25,6 +29,6 @@
             </command_interface>
             <state_interface name="position"/> <!-- <param name="initial_value">1.0</param> -->
-            <state_interface name="velocity"/>
-            <state_interface name="effort"/>
+            <!-- <state_interface name="velocity"/>
+            <state_interface name="effort"/> -->
         </joint>
         <joint name="joint3_to_joint2">
@@ -63,4 +67,48 @@
             <state_interface name="position"/>
         </joint>
+    </ros2_control>
+    <gazebo>
+      <!-- filename="gz_ros2_control-system" -->
+      <!-- <plugin filename="libgz_ros2_control-system" name="gz_ros2_control::GazeboSimROS2ControlPlugin"> -->
+      <plugin filename="gz_ros2_control-system" name="gz_ros2_control::GazeboSimROS2ControlPlugin">
+          <!--<robot_sim_type>gazebo_ros2_control/DefaultRobotHWSim</robot_sim_type> -->
+          <!-- A YAML file with the configuration of the controllers. This element can be given multiple times to load multiple files. -->
+          <parameters>$(find mycobot_description)/config/simple_controller.yaml</parameters>
+          <!-- one can specify a namespace and remapping rules, which will be forwarded to the controller_manager and loaded controllers -->
+          <ros>
+              <!-- <namespace>my_namespace</namespace> -->
+              <remapping>/controller_manager/robot_description:=/robot_description</remapping>
+          </ros>
+          <!-- The location of the robot_description (URDF) on the parameter server, defaults to robot_description-->
+          <!-- <robot_param>robot_description</robot_param> -->
+          <!-- Name of the node where the robot_param is located, defaults to robot_state_publisher -->
+          <!-- <robot_param_node>robot_state_publisher</robot_param_node>  -->
+          <!-- Set controller manager name -->
+          <!-- <controller_manager_name>controller_manager</controller_manager_name>  -->
+          <!-- set the controller manager node name -->
+          <!-- <controller_manager_prefix_node_name> </controller_manager_prefix_node_name>  -->
+      </plugin>
+  </gazebo>
+</robot>
+        <!-- I found in /opt/iron/ - could use this
+        ./lib/libjoint_trajectory_controller.so
+        ./lib/libjoint_state_broadcaster.so
+        ./lib/librobot_state_publisher_node.so
+        Could use them as: (but not needed since ros2_control will  handle)
+        /joint_states (from joint_state_publisher)
+          <gazebo>
+            <plugin filename="libjoint_state_broadcaster.so" name="Gazebo::systems::JointStateBroadCaster">
+                <topic>joint_states</topic>
+            </plugin>
+        </gazebo>
+        <gazebo>
+            <plugin filename="libjoint_trajectory_controller.so" name="Gazebo::systems::JointTrajectoryController">
+                <joint_name>joint6_to_joint5</joint_name>
+                <joints>joint2_to_joint1, joint3_to_joint2, joint4_to_joint3, joint5_to_joint4, joint6_to_joint5, joint6output_to_joint6 </joints>
+                <publish_selected_only>1</publish_selected_only>
+            </plugin>
+        </gazebo>
+        joint_pose_trajectory plugin for controlling
+        -->
         <!--  <joint name="gripper_controller">
             <command_interface name="position">
@@ -121,26 +169,2 @@
             <state_interface name="velocity"/>
         </joint> -->
-    </ros2_control>
-    <gazebo>
-      <!-- filename="gz_ros2_control-system" -->
-      <!-- <plugin filename="libgz_ros2_control-system" name="gz_ros2_control::GazeboSimROS2ControlPlugin"> -->
-      <plugin filename="gz_ros2_control-system" name="gz_ros2_control::GazeboSimROS2ControlPlugin">
-          <!--<robot_sim_type>gazebo_ros2_control/DefaultRobotHWSim</robot_sim_type> -->
-          <parameters>$(find mycobot_description)/config/simple_controller.yaml</parameters> <!-- A YAML file with the configuration of the controllers. This element can be given multiple times to load multiple files. -->
-          <!-- one can specify a namespace and remapping rules, which will be forwarded to the controller_manager and loaded controllers -->
-          <ros>
-              <!-- <namespace>my_namespace</namespace> -->
-              <remapping>/controller_manager/robot_description:=/robot_description</remapping>
-          </ros>
-          <!-- The location of the robot_description (URDF) on the parameter server, defaults to robot_description-->
-          <!-- <robot_param>robot_description</robot_param> -->
-          <!-- Name of the node where the robot_param is located, defaults to robot_state_publisher -->
-          <!-- <robot_param_node>robot_state_publisher</robot_param_node>  -->
-          <!-- Set controller manager name -->
-          <!-- <controller_manager_name>controller_manager</controller_manager_name>  -->
-          <!-- set the controller manager node name -->
-          <!-- <controller_manager_prefix_node_name> </controller_manager_prefix_node_name>  -->
-      </plugin>
-  </gazebo>
-  </xacro:macro>
-</robot>

File: my_project/src/mycobot_description/xacro/macro.gazebo_internal_config.xacro (robot description, xacro)
@@ -1,121 +1,45 @@
 <?xml version="1.0"?>
 <robot xmlns:xacro="http://www.ros.org/wiki/xacro">
-	<xacro:macro name="dsr_config_coeff">
     <!-- I need this for a better simulation in Gazebo-->
     <!-- Based on this https://github.com/dvalenciar/robotic_arm_environment/blob/main/my_doosan_pkg/description/xacro/macro.internal_config.xacro -->
     <!-- and this https://github.com/automaticaddison/mycobot_ros2/blob/main/mycobot_gazebo/urdf/ros2_control/gazebo/mycobot_280.urdf.xacro#L356-->
+    <!-- Check this for material colors: https://github.com/gazebosim/gazebo-classic/blob/d0c34b8a5d6bc9a3271000fb1baeb3f8d9f43afa/media/materials/scripts/gazebo.material-->
+    <!--Check this for Gazebo tags http://sdformat.org/tutorials?tut=sdformat_urdf_extensions&cat=specification& -->
+    <!-- ruby $(which gz) sim-4] [Wrn] [SdfEntityCreator.cc:824] Using an internal gazebo.material to parse Gazebo/Indigo
+[ruby $(which gz) sim-4] [Wrn] [SdfEntityCreator.cc:808] Gazebo does not support Ogre material scripts. See https://gazebosim.org/api/sim/8/migrationsdf.html#:~:text=Materials for details -->
     <!-- Base -->
     <gazebo reference="base_link">
-      <kp>1000000.0</kp>
+      <material>Gazebo/Blue</material>
+      <!-- <material name="blue"/> doesn't work-->
+    </gazebo>
+    <!-- Link1 -->
+    <gazebo reference="link1">
+      <material>Gazebo/Yellow</material>
+    </gazebo>
+    <!-- Link2 -->
+    <gazebo reference="link2">
+      <material>Gazebo/SkyBlue</material>
+    </gazebo>
+    <!-- Link3 -->
+    <gazebo reference="link3">
+      <material>Gazebo/ZincYellow</material>
+    </gazebo>
+    <!-- Link4 -->
+    <gazebo reference="link4">
+      <material>Gazebo/Turquoise</material>
+    </gazebo>
+    <!-- Link5 -->
+    <gazebo reference="link5">
+      <material>Gazebo/Indigo</material>
+    </gazebo>
+    <!-- Link6 -->
+    <gazebo reference="link6">
+      <!-- <kp>1000000.0</kp>
       <kd>100.0</kd>
       <mu1>30.0</mu1>
       <mu2>30.0</mu2>
       <maxVel>1.0</maxVel>
-      <minDepth>0.001</minDepth>
-      <!-- No support Ogre materialfiles like Classic does https://gazebosim.org/api/sim/8/migrationsdf.html#:~:text=Materials -->
-      <!-- <visual>
-        <material>
-        <ambient>0.5 0.5 0.5 1</ambient>
-        <diffuse>0.5 0.5 0.5 1</diffuse>
-        <specular>0.5 0.5 0.5 1</specular>
-        </material>
-      </visual> -->
+      <minDepth>0.001</minDepth> -->
+      <material>Gazebo/BlueGlow</material>
     </gazebo>
-    <!-- Link1 -->
-    <gazebo reference="link1">
-      <kp>1000000.0</kp>
-      <kd>100.0</kd>
-      <mu1>30.0</mu1>
-      <mu2>30.0</mu2>
-      <maxVel>1.0</maxVel>
-      <minDepth>0.001</minDepth>
-      <!-- <visual>
-        <material>
-          <ambient>0.5 0.5 0.5 1</ambient>
-          <diffuse>0.5 0.5 0.5 1</diffuse>
-          <specular>0.5 0.5 0.5 1</specular>
-        </material>
-      </visual> -->
-    </gazebo>
-    <!-- Link2 -->
-    <gazebo reference="link2">
-      <kp>1000000.0</kp>
-      <kd>100.0</kd>
-      <mu1>30.0</mu1>
-      <mu2>30.0</mu2>
-      <maxVel>1.0</maxVel>
-      <minDepth>0.001</minDepth>
-      <!-- <visual>
-        <material>
-          <ambient>1 1 1 1</ambient>
-          <diffuse>1 1 1 1</diffuse>
-          <specular>1 1 1 1</specular>
-        </material>
-      </visual> -->
-    </gazebo>
-    <!-- Link3 -->
-    <gazebo reference="link3">
-      <kp>1000000.0</kp>
-      <kd>100.0</kd>
-      <mu1>30.0</mu1>
-      <mu2>30.0</mu2>
-      <maxVel>1.0</maxVel>
-      <minDepth>0.001</minDepth>
-      <!-- <visual>
-        <material>
-          <ambient>1 1 1 1</ambient>
-          <diffuse>1 1 1 1</diffuse>
-          <specular>1 1 1 1</specular>
-        </material>
-      </visual> -->
-    </gazebo>
-    <!-- Link4 -->
-    <gazebo reference="link4">
-      <kp>1000000.0</kp>
-      <kd>100.0</kd>
-      <mu1>30.0</mu1>
-      <mu2>30.0</mu2>
-      <maxVel>1.0</maxVel>
-      <minDepth>0.001</minDepth>
-      <!-- <visual>
-        <material>
-          <ambient>1 1 1 1</ambient>
-          <diffuse>1 1 1 1</diffuse>
-          <specular>1 1 1 1</specular>
-        </material>
-      </visual> -->
-    </gazebo>
-    <!-- Link5 -->
-    <gazebo reference="link5">
-      <kp>1000000.0</kp>
-      <kd>100.0</kd>
-      <mu1>30.0</mu1>
-      <mu2>30.0</mu2>
-      <maxVel>1.0</maxVel>
-      <minDepth>0.001</minDepth>
-      <!-- <visual>
-        <material>
-          <ambient>1 1 1 1</ambient>
-          <diffuse>1 1 1 1</diffuse>
-          <specular>1 1 1 1</specular>
-        </material>
-      </visual> -->
-    </gazebo>
-    <!-- Link6 -->
-    <gazebo reference="link6">
-      <kp>1000000.0</kp>
-      <kd>100.0</kd>
-      <mu1>30.0</mu1>
-      <mu2>30.0</mu2>
-      <maxVel>1.0</maxVel>
-      <minDepth>0.001</minDepth>
-      <!-- <visual>
-        <material>
-          <ambient>1 1 1 1</ambient>
-          <diffuse>1 1 1 1</diffuse>
-          <specular>1 1 1 1</specular>
-        </material>
-      </visual> -->
-    </gazebo>
-	</xacro:macro>
 </robot>

File: my_project/src/mycobot_description/xacro/macro.mycobot_320_pi_2022.xacro (robot description, xacro)
@@ -7,4 +7,19 @@
   <xacro:include filename="$(find mycobot_description)/xacro/macro.gazebo_config_ros2_control.xacro" />
   <xacro:macro name="mycobot_320pi" params="namespace">
+    <material name="white">
+      <color rgba="1 1 1 1" />
+    </material>
+    <material name="orange">
+      <color rgba="1 0.3 0.1 1"/>
+    </material>
+    <material name="blue">
+      <color rgba="0.2 0.2 1 1"/>
+    </material>
+    <material name="black">
+      <color rgba="0 0 0 1"/>
+    </material>
+    <material name="red">
+      <color rgba="1 0 0 1"/>
+    </material>
     <!-- Base -->
     <link name="base_link">
@@ -25,4 +40,13 @@
           <mesh filename="file:///$(find mycobot_description)/mesh/base_link.dae" />
         </geometry>
+        <material name="violet"> <!-- default colors -  overriden by gazebo config-->
+          <color rgba="0.4 0.18 0.57 1.0" />
+        </material>
+          <!-- No support Ogre materialfiles like Classic does https://gazebosim.org/api/sim/8/migrationsdf.html#:~:text=Materials -->
+          <!-- <material>
+            <ambient>0.5 0.5 0.5 1</ambient>
+            <diffuse>0.5 0.5 0.5 1</diffuse>
+            <specular>0.5 0.5 0.5 1</specular>
+          </material> -->
       </visual>
       <collision>
@@ -49,4 +73,5 @@
           <mesh filename="file:///$(find mycobot_description)/mesh/link1.dae"/>
         </geometry>
+       <!-- <material name="orange"/> -->
       </visual>
       <collision>
@@ -72,4 +97,5 @@
           <mesh filename="file:///$(find mycobot_description)/mesh/link2.dae"/>
         </geometry>
+        <material name="black"/>
       </visual>
       <collision>
@@ -95,4 +121,5 @@
           <mesh filename="file:///$(find mycobot_description)/mesh/link3.dae"/>
         </geometry>
+        <material name="red"/>
       </visual>
       <collision>
@@ -118,4 +145,5 @@
           <mesh filename="file:///$(find mycobot_description)/mesh/link4.dae"/>
         </geometry>
+        <material name="black"/>
       </visual>
       <collision>
@@ -147,4 +175,5 @@
           <mesh filename="file:///$(find mycobot_description)/mesh/link5.dae"/>
         </geometry>
+        <material name="white"/>
       </collision>
     </link>
@@ -164,4 +193,5 @@
           <mesh filename="file:///$(find mycobot_description)/mesh/link6.dae"/>
         </geometry>
+        <material name="red"/>
       </visual>
       <collision>
